Commit message: added biotac stls, updated urdf path but still wrong

File: models/hand-model.urdf (robot description, URDF)
Before this commit: robot lbr4, 36 links, 35 joints
Links:
- link allegro_mount: geometry collision mesh filename=../models/allegro_model/allegro_mount.stl; visual mesh filename=../models/allegro_model/allegro_mount.stl
- link index_biotac_nail: geometry collision mesh filename=../models/allegro_model/biotac/nail_collision.stl; visual mesh filename=../models/allegro_model/biotac/nail_visual.stl
- link index_biotac_tip: geometry collision mesh filename=../models/allegro_model/biotac/contact_collision_small.stl; visual mesh filename=../models/allegro_model/biotac/contact_visual.stl
- link index_link_0: geometry collision mesh filename=../models/allegro_model/collision/link_0.0.stl; visual mesh filename=../models/allegro_model/link_0.0.stl
- link index_link_1: geometry collision mesh filename=../models/allegro_model/collision/link_1.0.stl; visual mesh filename=../models/allegro_model/allegro/link_1.0.stl
- link index_link_2: geometry collision mesh filename=../models/allegro_model/collision/link_2.0.stl; visual mesh filename=../models/allegro_model/link_2.0.stl
- link index_link_3: geometry collision mesh filename=../models/allegro_model/collision/link_3.0.stl; visual mesh filename=../models/allegro_model/link_3.0.stl
- link index_tip: geometry collision mesh filename=../models/allegro_model/biotac/base_collision.stl; visual mesh filename=../models/allegro_model/biotac/base_visual.stl
- link middle_biotac_nail: geometry collision mesh filename=../models/allegro_model/biotac/nail_collision.stl; visual mesh filename=../models/allegro_model/biotac/nail_visual.stl
- link middle_biotac_tip: geometry collision mesh filename=../models/allegro_model/biotac/contact_collision_small.stl; visual mesh filename=../models/allegro_model/biotac/contact_visual.stl
- link middle_link_0: geometry collision mesh filename=../models/allegro_model/collision/link_0.0.stl; visual mesh filename=../models/allegro_model/link_0.0.stl
- link middle_link_1: geometry collision mesh filename=../models/allegro_model/collision/link_1.0.stl; visual mesh filename=../models/allegro_model/link_1.0.stl
- link middle_link_2: geometry collision mesh filename=../models/allegro_model/collision/link_2.0.stl; visual mesh filename=../models/allegro_model/link_2.0.stl
- link middle_link_3: geometry collision mesh filename=../models/allegro_model/collision/link_3.0.stl; visual mesh filename=../models/allegro_model/link_3.0.stl
- link middle_tip: geometry collision mesh filename=../models/allegro_model/biotac/base_collision.stl; visual mesh filename=../models/allegro_model/biotac/base_visual.stl
- link palm_link: geometry collision mesh filename=../models/allegro_model/collision/base_link_biotac.stl; visual mesh filename=../models/allegro_model/base_link_biotac.stl
- link ring_biotac_nail: geometry collision mesh filename=../models/allegro_model/biotac/nail_collision.stl; visual mesh filename=../models/allegro_model/biotac/nail_visual.stl
- link ring_biotac_tip: geometry collision mesh filename=../models/allegro_model/biotac/contact_collision_small.stl; visual mesh filename=../models/allegro_model/biotac/contact_visual.stl
- link ring_link_0: geometry collision mesh filename=../models/allegro_model/collision/link_0.0.stl; visual mesh filename=../models/allegro_model/link_0.0.stl
- link ring_link_1: geometry collision mesh filename=../models/allegro_model/collision/link_1.0.stl; visual mesh filename=../models/allegro_model/link_1.0.stl
- link ring_link_2: geometry collision mesh filename=../models/allegro_model/collision/link_2.0.stl; visual mesh filename=../models/allegro_model/link_2.0.stl
- link ring_link_3: geometry collision mesh filename=../models/allegro_model/collision/link_3.0.stl; visual mesh filename=../models/allegro_model/link_3.0.stl
- link ring_tip: geometry collision mesh filename=../models/allegro_model/biotac/base_collision.stl; visual mesh filename=../models/allegro_model/biotac/base_visual.stl
- link thumb_biotac_nail: geometry collision mesh filename=../models/allegro_model/biotac/nail_collision.stl; visual mesh filename=../models/allegro_model/biotac/nail_visual.stl
- link thumb_biotac_tip: geometry collision mesh filename=../models/allegro_model/biotac/contact_collision_small.stl; visual mesh filename=../models/allegro_model/biotac/contact_visual.stl
- link thumb_link_0: geometry collision mesh filename=../models/allegro_model/collision/link_12.0_right.stl; visual mesh filename=../models/allegro_model/link_12.0_right.stl
- link thumb_link_1: geometry collision mesh filename=../models/allegro_model/collision/link_13.0.stl; visual mesh filename=../models/allegro_model/link_13.0.stl
- link thumb_link_2: geometry collision mesh filename=../models/allegro_model/collision/link_14.0.stl; visual mesh filename=../models/allegro_model/link_14.0.stl
- link thumb_link_3: geometry collision mesh filename=../models/allegro_model/collision/link_15.0.stl; visual mesh filename=../models/allegro_model/link_15.0.stl
- link thumb_tip: geometry collision mesh filename=../models/allegro_model/biotac/base_collision.stl; visual mesh filename=../models/allegro_model/biotac/base_visual.stl

Commit message: fixed fiepaths

File: models/hand-model.urdf (robot description, URDF)
Before this commit: robot lbr4, 36 links, 35 joints
Links:
- link index_link_1: geometry collision mesh filename=../models/allegro_model/collision/link_1.0.stl; visual mesh filename=../models/allegro_model/link_1.0.stl
